File: miwos.brd (EAGLE design)
At the start: 120 x 120 mm, 44 parts, among them J1 614004190021, U1 PEC16, U3 PEC16

Commit message: Use lorenz's version
Parts:
- moved R11 57.3 mm to (43.2, 105.4)
- moved R9 44.7 mm to (40.6, 96.5)
- moved C2 43.7 mm to (73.7, 80.0)
- moved R1 21.1 mm to (90.2, 88.9), turned to 180 degrees
- moved D2 19.7 mm to (79.9, 94.2), turned to 180 degrees
- moved R4 19.1 mm to (94.0, 82.5), turned to 180 degrees
- moved R10 18.3 mm to (45.7, 63.5), turned to 270 degrees
- moved R2 17.0 mm to (86.4, 82.5), turned to 180 degrees
- moved D1 15.9 mm to (33.0, 69.8)
- moved R3 13.2 mm to (86.4, 85.7), turned to 180 degrees
- moved R8 13.1 mm to (29.2, 67.3)
- moved OK1 3.59 mm to (77.5, 86.4), turned to 90 degrees
- moved TEENSY-41 1.67 mm to (59.7, 86.4)
- moved C1 1.27 mm to (43.2, 69.8)
Routing:
- net SCL-1: track 117.0 -> 51.7 mm, vias 0 -> 2
- net N$12: track 70.1 -> 5.27 mm
- net N$11: track 64.9 -> 6.31 mm
- net TX-5: track 71.1 -> 13.6 mm
- net +5V: track 184.9 -> 130.5 mm, vias 0 -> 2
- net SDA-1: track 104.4 -> 53.3 mm, vias 0 -> 2
- net RX-2: track 76.7 -> 25.7 mm
- net N$19: track 32.7 -> 2.01 mm
- net N$18: track 37.1 -> 12.4 mm
- net N$21: track 26.0 -> 4.61 mm
- net RX-5: track 76.2 -> 56.0 mm
- net N$17: track 32.7 -> 16.2 mm
- net N$3: track 102.8 -> 87.1 mm
- net N$10: track 48.5 -> 34.0 mm
- net BUTTON-4: track 58.4 -> 45.4 mm
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- added copper zone on layer 1, net GND
- added copper zone on layer 16, net GND

Commit message: Wire encoders
Parts:
- moved R6 139.8 mm to (-34.4, 24.0)
- moved LED2 138.0 mm to (-33.2, 30.3)
- moved R5 137.0 mm to (-24.1, 23.1)
- moved LED1 135.8 mm to (-23.5, 30.8)
- moved LED3 124.3 mm to (-24.7, 3.86)
- moved R7 122.5 mm to (-25.3, 8.67)
- moved R14 95.3 mm to (-12.7, 8.89)
- moved LED6 88.9 mm to (-11.8, 4.27)
- moved R13 86.4 mm to (-20.3, 8.89)
- moved R12 80.0 mm to (-31.8, 8.89)
- moved LED5 78.1 mm to (-17.8, 3.81)
- moved LED4 75.0 mm to (-31.6, 3.07)
- moved S2 1.84 mm to (90.2, 61.0)
- moved R10 1.27 mm to (45.7, 62.2), turned to 180 degrees
- moved TEENSY-41 1.27 mm to (59.7, 87.6)
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Connections:
- net BUTTON-1-LED: no longer TEENSY-41.28
- net BUTTON-2: now also TEENSY-41.28; no longer TEENSY-41.29
- net BUTTON-2-LED: no longer TEENSY-41.30
- net BUTTON-3: now also TEENSY-41.29; no longer TEENSY-41.31/A12
- net BUTTON-3-LED: no longer TEENSY-41.32
- net BUTTON-4: now also TEENSY-41.30; no longer TEENSY-41.33
- net BUTTON-4-LED: no longer TEENSY-41.34
- net BUTTON-5: now also TEENSY-41.31/A12; no longer TEENSY-41.35
- net BUTTON-5-LED: no longer TEENSY-41.36
- net BUTTON-6: now also TEENSY-41.32; no longer TEENSY-41.37
- net BUTTON-6-LED: no longer TEENSY-41.38
- net ENCODER-1-A: now also TEENSY-41.2
- net ENCODER-1-B: now also TEENSY-41.3
- net ENCODER-1-PUSH: now also TEENSY-41.23/A9
- net ENCODER-2-A: now also TEENSY-41.37
- net ENCODER-2-B: now also TEENSY-41.36
- net ENCODER-2-PUSH: now also TEENSY-41.38
- net ENCODER-3-A: now also TEENSY-41.34
- net ENCODER-3-B: now also TEENSY-41.33
- net ENCODER-3-PUSH: now also TEENSY-41.35
Routing:
- net BUTTON-6-LED: track 75.2 -> 0.00 mm
- net ENCODER-1-A: track 0.00 -> 65.2 mm
- net BUTTON-5-LED: track 64.7 -> 0.00 mm
- net BUTTON-4-LED: track 59.7 -> 0.00 mm
- net ENCODER-1-B: track 0.00 -> 53.4 mm
- net ENCODER-3-A: track 0.00 -> 51.5 mm
- net ENCODER-2-A: track 0.00 -> 50.1 mm
- net ENCODER-2-PUSH: track 0.00 -> 40.3 mm
- net ENCODER-3-B: track 0.00 -> 39.7 mm
- net ENCODER-2-B: track 0.00 -> 38.3 mm
- net BUTTON-1-LED: track 37.7 -> 0.00 mm
- net BUTTON-2-LED: track 35.5 -> 0.00 mm
- net ENCODER-1-PUSH: track 0.00 -> 31.7 mm
- net ENCODER-3-PUSH: track 0.00 -> 28.3 mm
- net BUTTON-3-LED: track 28.2 -> 0.00 mm
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
Commit message: Small fixes
Parts:
- moved R11 1.27 mm to (41.9, 105.4)
Routing:
- net N$2: track 85.6 -> 92.5 mm
- net +3V3: track 172.1 -> 173.4 mm
- net N$3: track 88.4 -> 87.7 mm
- net N$12: track 5.27 -> 5.80 mm
Changed lines of the file:
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@@
 <setting verticaltext="up"/>
 </settings>
-<grid distance="50" unitdist="mil" unit="mil" style="lines" multiple="1" display="yes" altdistance="1" altunitdist="mil" altunit="mil"/>
+<grid distance="50" unitdist="mil" unit="mil" style="lines" multiple="1" display="yes" altdistance="25" altunitdist="mil" altunit="mil"/>
 <layers>
 <layer number="1" name="Top" color="4" fill="1" visible="yes" active="yes"/>
@@
 <attribute name="VALUE" x="46.355" y="64.135" size="1.27" layer="27" rot="R180"/>
 </element>
-<element name="R11" library="rcl" library_urn="urn:adsk.eagle:library:334" package="R0603" package3d_urn="urn:adsk.eagle:package:23555/3" value="47R" x="43.18" y="105.41" smashed="yes">
-<attribute name="NAME" x="42.545" y="106.045" size="1.27" layer="25"/>
-<attribute name="POPULARITY" value="70" x="-17.78" y="123.19" size="1.778" layer="27" display="off"/>
-<attribute name="SPICEPREFIX" value="R" x="-17.78" y="123.19" size="1.778" layer="27" display="off"/>
-<attribute name="VALUE" x="42.545" y="103.505" size="1.27" layer="27"/>
+<element name="R11" library="rcl" library_urn="urn:adsk.eagle:library:334" package="R0603" package3d_urn="urn:adsk.eagle:package:23555/3" value="47R" x="41.91" y="105.41" smashed="yes">
+<attribute name="NAME" x="41.275" y="106.045" size="1.27" layer="25"/>
+<attribute name="POPULARITY" value="70" x="-19.05" y="123.19" size="1.778" layer="27" display="off"/>
+<attribute name="SPICEPREFIX" value="R" x="-19.05" y="123.19" size="1.778" layer="27" display="off"/>
+<attribute name="VALUE" x="41.275" y="103.505" size="1.27" layer="27"/>
 </element>
 <element name="C1" library="rcl" library_urn="urn:adsk.eagle:library:334" package="C0603" package3d_urn="urn:adsk.eagle:package:23616/2" value="0.1uF" x="43.18" y="69.85" smashed="yes">
@@
 <wire x1="86.995" y1="82.335" x2="87.21" y2="82.55" width="0.4064" layer="1"/>
 <wire x1="86.995" y1="82.335" x2="86.995" y2="78.105" width="0.4064" layer="1"/>
-<wire x1="44.03" y1="105.41" x2="50.38" y2="111.76" width="0.4064" layer="1"/>
+<wire x1="42.76" y1="105.41" x2="44.03" y2="105.41" width="0.4064" layer="1"/>
 <wire x1="50.38" y1="111.76" x2="52.07" y2="111.76" width="0.4064" layer="1"/>
 <wire x1="48.75" y1="35.16" x2="45.51" y2="38.4" width="0.4064" layer="1"/>
@@
 <wire x1="46.57" y1="62.23" x2="46.99" y2="61.81" width="0.4064" layer="1"/>
 <wire x1="46.99" y1="61.81" x2="46.99" y2="57.36" width="0.4064" layer="1"/>
+<wire x1="44.03" y1="105.41" x2="50.38" y2="111.76" width="0.4064" layer="1"/>
 <wire x1="67.31" y1="81.28" x2="48.26" y2="82.55" width="0" layer="19" extent="1-1"/>
 </signal>
@@
 <wire x1="111.0142" y1="61.3572" x2="105.9038" y2="61.3572" width="0.254" layer="1"/>
 <wire x1="114.3" y1="64.643" x2="111.0142" y2="61.3572" width="0.254" layer="1"/>
-<wire x1="108.4957375" y1="80.7342625" x2="114.3" y2="74.93" width="0.254" layer="1"/>
-<wire x1="103.96669375" y1="85.26330625" x2="103.96669375" y2="81.96130625" width="0.254" layer="1"/>
-<wire x1="105.1937375" y1="80.7342625" x2="108.4957375" y2="80.7342625" width="0.254" layer="1"/>
-<wire x1="103.96669375" y1="81.96130625" x2="105.1937375" y2="80.7342625" width="0.254" layer="1"/>
-<wire x1="64.31" y1="107.95" x2="65.6562" y2="106.6038" width="0.254" layer="1"/>
-<wire x1="82.6262" y1="106.6038" x2="65.6562" y2="106.6038" width="0.254" layer="1"/>
-<wire x1="82.6262" y1="106.6038" x2="103.96669375" y2="85.26330625" width="0.254" layer="1"/>
+<wire x1="109.22" y1="80.01" x2="114.3" y2="74.93" width="0.254" layer="1"/>
+<wire x1="77.5462" y1="111.6838" x2="74.93" y2="111.6838" width="0.254" layer="1"/>
+<wire x1="77.5462" y1="111.6838" x2="84.455" y2="104.775" width="0.254" layer="1"/>
+<wire x1="102.87" y1="86.36" x2="92.71" y2="96.52" width="0.254" layer="1"/>
+<wire x1="84.455" y1="104.775" x2="90.805" y2="104.775" width="0.254" layer="1"/>
+<wire x1="90.805" y1="104.775" x2="92.71" y2="102.87" width="0.254" layer="1"/>
+<wire x1="92.71" y1="102.87" x2="92.71" y2="96.52" width="0.254" layer="1"/>
+<wire x1="102.87" y1="86.36" x2="106.32339375" y2="86.36" width="0.254" layer="1"/>
+<wire x1="106.32339375" y1="86.36" x2="109.22" y2="83.46339375" width="0.254" layer="1"/>
+<wire x1="109.22" y1="83.46339375" x2="109.22" y2="80.01" width="0.254" layer="1"/>
+<wire x1="74.93" y1="111.6838" x2="71.1962" y2="107.95" width="0.254" layer="1"/>
+<wire x1="71.1962" y1="107.95" x2="64.31" y2="107.95" width="0.254" layer="1"/>
 </signal>
 <signal name="N$3">
 <contactref element="J1" pad="3"/>
 <contactref element="TEENSY-41" pad="UD+"/>
-<wire x1="82.0166" y1="105.9434" x2="70.3834" y2="105.9434" width="0.254" layer="1"/>
-<wire x1="102.87" y1="85.09" x2="82.0166" y2="105.9434" width="0.254" layer="1"/>
+<wire x1="70.485" y1="106.045" x2="81.915" y2="106.045" width="0.254" layer="1"/>
+<wire x1="102.87" y1="85.09" x2="81.915" y2="106.045" width="0.254" layer="1"/>
 <wire x1="113.03" y1="74.93" x2="107.95" y2="80.01" width="0.254" layer="1"/>
 <wire x1="113.03" y1="64.5784" x2="113.03" y2="74.93" width="0.254" layer="1"/>
 <wire x1="64.31" y1="105.41" x2="69.85" y2="105.41" width="0.254" layer="1"/>
-<wire x1="69.85" y1="105.41" x2="70.3834" y2="105.9434" width="0.254" layer="1"/>
+<wire x1="69.85" y1="105.41" x2="70.485" y2="106.045" width="0.254" layer="1"/>
 <wire x1="105.9038" y1="59.3572" x2="104.4728" y2="59.3572" width="0.254" layer="1"/>
 <wire x1="104.4728" y1="59.3572" x2="104.14" y2="59.69" width="0.254" layer="1"/>
@@
 <wire x1="111.3166" y1="62.865" x2="113.03" y2="64.5784" width="0.254" layer="1"/>
 <wire x1="106.31648125" y1="62.865" x2="111.3166" y2="62.865" width="0.254" layer="1"/>
-<wire x1="107.95" y1="80.01" x2="104.648" y2="80.01" width="0.254" layer="1"/>
-<wire x1="104.648" y1="80.01" x2="102.87" y2="81.788" width="0.254" layer="1"/>
-<wire x1="102.87" y1="81.788" x2="102.87" y2="85.09" width="0.254" layer="1"/>
+<wire x1="107.95" y1="80.01" x2="105.918" y2="80.01" width="0.254" layer="1"/>
+<wire x1="105.918" y1="80.01" x2="102.87" y2="83.058" width="0.254" layer="1"/>
+<wire x1="102.87" y1="83.058" x2="102.87" y2="85.09" width="0.254" layer="1"/>
 </signal>
 <signal name="BUTTON-1">
@@
 <contactref element="R11" pad="1"/>
 <contactref element="MIDI-OUT-2" pad="4"/>
-<wire x1="42.33" y1="105.41" x2="42.33" y2="104.99" width="0.254" layer="1"/>
-<wire x1="44.7463875" y1="101.139515625" x2="44.7463875" y2="102.5736125" width="0.254" layer="1"/>
-<wire x1="44.7463875" y1="102.5736125" x2="42.33" y2="104.99" width="0.254" layer="1"/>
+<wire x1="44.7463875" y1="101.139515625" x2="44.7463875" y2="101.3036125" width="0.254" layer="1"/>
+<wire x1="44.7463875" y1="101.3036125" x2="41.06" y2="104.99" width="0.254" layer="1"/>
+<wire x1="41.06" y1="105.41" x2="41.06" y2="104.99" width="0.254" layer="1"/>
 </signal>
 <signal name="N$13">

Commit message: Refactor, add button LEDs
Parts:
- moved R6 138.3 mm to (97.8, 64.8)
- moved LED2 137.1 mm to (100.3, 61.0)
- moved LED1 136.2 mm to (105.4, 74.9)
- moved R5 135.7 mm to (102.9, 71.1)
- moved LED3 123.6 mm to (90.2, 49.5)
- moved R7 121.4 mm to (87.6, 53.3)
- moved LED6 89.3 mm to (77.5, 6.35)
- moved R14 85.1 mm to (72.4, 6.35)
- moved R12 80.1 mm to (48.3, 6.35), turned to 180 degrees
- moved LED5 77.5 mm to (59.7, 6.35)
- moved R13 75.0 mm to (54.6, 6.35)
- moved LED4 74.8 mm to (43.2, 6.35), turned to 180 degrees
Connections:
- new net N$1: TEENSY-41.39
- net BUTTON-1-LED: now also TEENSY-41.10/CS
- net BUTTON-2-LED: now also TEENSY-41.11/MOSI
- net BUTTON-3-LED: now also TEENSY-41.12/MISO
- net BUTTON-4-LED: now also TEENSY-41.14/A0
- net BUTTON-5-LED: now also TEENSY-41.15/A1
- net BUTTON-6-LED: now also TEENSY-41.22/A8
Routing:
- net BUTTON-6-LED: track 0.00 -> 118.5 mm, vias 0 -> 2
- net BUTTON-5-LED: track 0.00 -> 85.0 mm, vias 0 -> 2
- net BUTTON-4-LED: track 0.00 -> 83.3 mm, vias 0 -> 2
- net BUTTON-1-LED: track 0.00 -> 49.1 mm, vias 0 -> 1
- net BUTTON-2-LED: track 0.00 -> 44.5 mm, vias 0 -> 1
- net BUTTON-3-LED: track 0.00 -> 40.8 mm, vias 0 -> 1
- net ENCODER-2-PUSH: track 40.3 -> 55.1 mm, vias 0 -> 1
- net BUTTON-6: track 49.2 -> 42.9 mm
- net ENCODER-1-A: track 65.2 -> 60.3 mm, vias 0 -> 3
- net N$7: track 0.00 -> 3.98 mm
- net N$5: track 0.00 -> 3.98 mm
- net N$6: track 0.00 -> 3.98 mm
- net N$15: track 0.00 -> 2.96 mm
- net N$14: track 0.13 -> 3.09 mm
- net N$13: track 0.00 -> 2.96 mm
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