File: miwos.sch (EAGLE design)
At the start: 44 parts, among them J1 614004190021, U1 PEC16, U3 PEC16

Commit message: Use lorenz's version
Other:
- moved on the sheet: R1, R9
Changed lines of the file:
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@@
 <attribute name="VALUE" x="131.8514" y="134.62" size="1.778" layer="96" rot="R90"/>
 </instance>
-<instance part="R1" gate="G$1" x="137.16" y="96.52" smashed="yes">
-<attribute name="NAME" x="133.35" y="98.0186" size="1.778" layer="95"/>
-<attribute name="VALUE" x="133.35" y="93.218" size="1.778" layer="96"/>
+<instance part="R1" gate="G$1" x="121.92" y="96.52" smashed="yes">
+<attribute name="NAME" x="118.11" y="98.0186" size="1.778" layer="95"/>
+<attribute name="VALUE" x="118.11" y="93.218" size="1.778" layer="96"/>
 </instance>
 <instance part="P+2" gate="1" x="160.02" y="154.94" smashed="yes">
@@
 <attribute name="VALUE" x="131.8514" y="66.04" size="1.778" layer="96" rot="R90"/>
 </instance>
-<instance part="R9" gate="G$1" x="137.16" y="27.94" smashed="yes">
-<attribute name="NAME" x="133.35" y="29.4386" size="1.778" layer="95"/>
-<attribute name="VALUE" x="133.35" y="24.638" size="1.778" layer="96"/>
+<instance part="R9" gate="G$1" x="121.92" y="27.94" smashed="yes">
+<attribute name="NAME" x="118.11" y="29.4386" size="1.778" layer="95"/>
+<attribute name="VALUE" x="118.11" y="24.638" size="1.778" layer="96"/>
 </instance>
 <instance part="P+3" gate="1" x="160.02" y="86.36" smashed="yes">
@@
 <pinref part="MIDI-OUT-1" gate="G$1" pin="5"/>
 <pinref part="R1" gate="G$1" pin="1"/>
-<wire x1="111.76" y1="96.52" x2="132.08" y2="96.52" width="0.1524" layer="91"/>
+<wire x1="111.76" y1="96.52" x2="116.84" y2="96.52" width="0.1524" layer="91"/>
 </segment>
 </net>
@@
 <pinref part="MIDI-OUT-2" gate="G$1" pin="5"/>
 <pinref part="R9" gate="G$1" pin="1"/>
-<wire x1="111.76" y1="27.94" x2="132.08" y2="27.94" width="0.1524" layer="91"/>
+<wire x1="111.76" y1="27.94" x2="116.84" y2="27.94" width="0.1524" layer="91"/>
 </segment>
 </net>
@@
 <segment>
 <pinref part="R1" gate="G$1" pin="2"/>
-<wire x1="142.24" y1="96.52" x2="147.32" y2="96.52" width="0.1524" layer="91"/>
+<wire x1="127" y1="96.52" x2="147.32" y2="96.52" width="0.1524" layer="91"/>
 <label x="149.86" y="96.52" size="1.778" layer="95"/>
 </segment>
@@
 <segment>
 <pinref part="R9" gate="G$1" pin="2"/>
-<wire x1="142.24" y1="27.94" x2="147.32" y2="27.94" width="0.1524" layer="91"/>
+<wire x1="127" y1="27.94" x2="147.32" y2="27.94" width="0.1524" layer="91"/>
 <label x="149.86" y="27.94" size="1.778" layer="95"/>
 </segment>

Commit message: Wire encoders
Connections:
- net BUTTON-1-LED: no longer TEENSY-41G$1.28
- net BUTTON-2: now also TEENSY-41G$1.28; no longer TEENSY-41G$1.29
- net BUTTON-2-LED: no longer TEENSY-41G$1.30
- net BUTTON-3: now also TEENSY-41G$1.29; no longer TEENSY-41G$1.31
- net BUTTON-3-LED: no longer TEENSY-41G$1.32
- net BUTTON-4: now also TEENSY-41G$1.30; no longer TEENSY-41G$1.33
- net BUTTON-4-LED: no longer TEENSY-41G$1.34
- net BUTTON-5: now also TEENSY-41G$1.31; no longer TEENSY-41G$1.35
- net BUTTON-5-LED: no longer TEENSY-41G$1.36
- net BUTTON-6: now also TEENSY-41G$1.32; no longer TEENSY-41G$1.37
- net BUTTON-6-LED: no longer TEENSY-41G$1.38
- net ENCODER-1-A: now also TEENSY-41G$1.2
- net ENCODER-1-B: now also TEENSY-41G$1.3
- net ENCODER-1-PUSH: now also TEENSY-41G$1.23
- net ENCODER-2-A: now also TEENSY-41G$1.37
- net ENCODER-2-B: now also TEENSY-41G$1.36
- net ENCODER-2-PUSH: now also TEENSY-41G$1.38
- net ENCODER-3-A: now also TEENSY-41G$1.34
- net ENCODER-3-B: now also TEENSY-41G$1.33
- net ENCODER-3-PUSH: now also TEENSY-41G$1.35
Changed lines of the file:
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@@
 <attribute name="VALUE" x="53.34" y="99.06" size="1.778" layer="96" rot="R90"/>
 </instance>
-<instance part="SUPPLY9" gate="GND" x="-17.78" y="81.28" smashed="yes">
-<attribute name="VALUE" x="-19.685" y="78.105" size="1.778" layer="96"/>
+<instance part="SUPPLY9" gate="GND" x="-20.32" y="81.28" smashed="yes">
+<attribute name="VALUE" x="-22.225" y="78.105" size="1.778" layer="96"/>
 </instance>
 <instance part="R3" gate="G$1" x="121.92" y="137.16" smashed="yes">
@@
 <segment>
 <pinref part="SUPPLY9" gate="GND" pin="GND"/>
-<wire x1="-17.78" y1="83.82" x2="-17.78" y2="91.44" width="0.1524" layer="91"/>
+<wire x1="-20.32" y1="83.82" x2="-20.32" y2="91.44" width="0.1524" layer="91"/>
 <pinref part="TEENSY-41" gate="G$1" pin="GND"/>
-<wire x1="-17.78" y1="91.44" x2="7.62" y2="91.44" width="0.1524" layer="91"/>
+<wire x1="-20.32" y1="91.44" x2="7.62" y2="91.44" width="0.1524" layer="91"/>
 </segment>
 <segment>
@@
 <label x="-88.9" y="40.64" size="1.778" layer="95" rot="R270"/>
 </segment>
+<segment>
+<pinref part="TEENSY-41" gate="G$1" pin="37"/>
+<wire x1="43.18" y1="43.18" x2="48.26" y2="43.18" width="0.1524" layer="91"/>
+<label x="50.8" y="43.18" size="1.778" layer="95"/>
+</segment>
 </net>
 <net name="ENCODER-3-B" class="0">
@@
 <wire x1="-81.28" y1="-22.86" x2="-81.28" y2="-25.4" width="0.1524" layer="91"/>
 <label x="-81.28" y="-27.94" size="1.778" layer="95" rot="R270"/>
+</segment>
+<segment>
+<pinref part="TEENSY-41" gate="G$1" pin="33"/>
+<wire x1="43.18" y1="33.02" x2="48.26" y2="33.02" width="0.1524" layer="91"/>
+<label x="50.8" y="33.02" size="1.778" layer="95"/>
 </segment>
 </net>
@@
 <label x="-88.9" y="104.14" size="1.778" layer="95" rot="R270"/>
 </segment>
+<segment>
+<pinref part="TEENSY-41" gate="G$1" pin="2"/>
+<wire x1="7.62" y1="83.82" x2="2.54" y2="83.82" width="0.1524" layer="91"/>
+<label x="-15.24" y="83.82" size="1.778" layer="95"/>
+</segment>
 </net>
 <net name="ENCODER-1-B" class="0">
@@
 <label x="-81.28" y="104.14" size="1.778" layer="95" rot="R270"/>
 </segment>
+<segment>
+<pinref part="TEENSY-41" gate="G$1" pin="3"/>
+<wire x1="7.62" y1="81.28" x2="2.54" y2="81.28" width="0.1524" layer="91"/>
+<label x="-15.24" y="81.28" size="1.778" layer="95"/>
+</segment>
 </net>
 <net name="ENCODER-1-PUSH" class="0">
@@
 <label x="-86.36" y="139.7" size="1.778" layer="95"/>
 </segment>
+<segment>
+<pinref part="TEENSY-41" gate="G$1" pin="23"/>
+<wire x1="43.18" y1="83.82" x2="48.26" y2="83.82" width="0.1524" layer="91"/>
+<label x="50.8" y="83.82" size="1.778" layer="95"/>
+</segment>
 </net>
 <net name="ENCODER-2-B" class="0">
@@
 <label x="-81.28" y="40.64" size="1.778" layer="95" rot="R270"/>
 </segment>
+<segment>
+<pinref part="TEENSY-41" gate="G$1" pin="36"/>
+<wire x1="43.18" y1="40.64" x2="48.26" y2="40.64" width="0.1524" layer="91"/>
+<label x="50.8" y="40.64" size="1.778" layer="95"/>
+</segment>
 </net>
 <net name="ENCODER-2-PUSH" class="0">
@@
 <label x="-86.36" y="73.66" size="1.778" layer="95"/>
 </segment>
+<segment>
+<pinref part="TEENSY-41" gate="G$1" pin="38"/>
+<wire x1="43.18" y1="45.72" x2="48.26" y2="45.72" width="0.1524" layer="91"/>
+<label x="50.8" y="45.72" size="1.778" layer="95"/>
+</segment>
 </net>
 <net name="ENCODER-3-A" class="0">
@@
 <label x="-88.9" y="-27.94" size="1.778" layer="95" rot="R270"/>
 </segment>
+<segment>
+<pinref part="TEENSY-41" gate="G$1" pin="34"/>
+<wire x1="43.18" y1="35.56" x2="48.26" y2="35.56" width="0.1524" layer="91"/>
+<label x="50.8" y="35.56" size="1.778" layer="95"/>
+</segment>
 </net>
 <net name="ENCODER-3-PUSH" class="0">
@@
 <label x="-86.36" y="10.16" size="1.778" layer="95"/>
 </segment>
+<segment>
+<pinref part="TEENSY-41" gate="G$1" pin="35"/>
+<wire x1="43.18" y1="38.1" x2="48.26" y2="38.1" width="0.1524" layer="91"/>
+<label x="50.8" y="38.1" size="1.778" layer="95"/>
+</segment>
 </net>
 <net name="N$2" class="0">
@@
 <pinref part="TEENSY-41" gate="G$1" pin="27"/>
 <wire x1="7.62" y1="45.72" x2="2.54" y2="45.72" width="0.1524" layer="91"/>
-<label x="-17.78" y="45.72" size="1.778" layer="95"/>
+<label x="-12.7" y="45.72" size="1.778" layer="95"/>
 </segment>
 </net>
@@
 </segment>
 <segment>
-<pinref part="TEENSY-41" gate="G$1" pin="29"/>
-<wire x1="7.62" y1="40.64" x2="2.54" y2="40.64" width="0.1524" layer="91"/>
-<label x="-17.78" y="40.64" size="1.778" layer="95"/>
+<pinref part="TEENSY-41" gate="G$1" pin="28"/>
+<wire x1="7.62" y1="43.18" x2="2.54" y2="43.18" width="0.1524" layer="91"/>
+<label x="-12.7" y="43.18" size="1.778" layer="95"/>
 </segment>
 </net>
@@
 </segment>
 <segment>
-<pinref part="TEENSY-41" gate="G$1" pin="31"/>
-<wire x1="7.62" y1="35.56" x2="2.54" y2="35.56" width="0.1524" layer="91"/>
-<label x="-17.78" y="35.56" size="1.778" layer="95"/>
+<pinref part="TEENSY-41" gate="G$1" pin="29"/>
+<wire x1="7.62" y1="40.64" x2="2.54" y2="40.64" width="0.1524" layer="91"/>
+<label x="-12.7" y="40.64" size="1.778" layer="95"/>
 </segment>
 </net>
@@
 <pinref part="R5" gate="G$1" pin="1"/>
 </segment>
-<segment>
-<pinref part="TEENSY-41" gate="G$1" pin="28"/>
-<wire x1="7.62" y1="43.18" x2="2.54" y2="43.18" width="0.1524" layer="91"/>
-<label x="-17.78" y="43.18" size="1.778" layer="95"/>
-</segment>
 </net>
 <net name="N$5" class="0">
@@
 <label x="20.32" y="-27.94" size="1.778" layer="95" rot="R180"/>
 </segment>
-<segment>
-<pinref part="TEENSY-41" gate="G$1" pin="30"/>
-<wire x1="7.62" y1="38.1" x2="2.54" y2="38.1" width="0.1524" layer="91"/>
-<label x="-17.78" y="38.1" size="1.778" layer="95"/>
-</segment>
 </net>
 <net name="N$6" class="0">
@@
 <pinref part="R7" gate="G$1" pin="1"/>
 <label x="73.66" y="-27.94" size="1.778" layer="95" rot="R180"/>
-</segment>
-<segment>
-<pinref part="TEENSY-41" gate="G$1" pin="32"/>
-<wire x1="7.62" y1="33.02" x2="2.54" y2="33.02" width="0.1524" layer="91"/>
-<label x="-17.78" y="33.02" size="1.778" layer="95"/>
 </segment>
 </net>
@@
 <pinref part="R12" gate="G$1" pin="1"/>
 </segment>
-<segment>
-<pinref part="TEENSY-41" gate="G$1" pin="34"/>
-<wire x1="43.18" y1="35.56" x2="48.26" y2="35.56" width="0.1524" layer="91"/>
-<label x="50.8" y="35.56" size="1.778" layer="95"/>
-</segment>
 </net>
 <net name="BUTTON-4" class="0">
@@
 </segment>
 <segment>
-<pinref part="TEENSY-41" gate="G$1" pin="33"/>
-<wire x1="43.18" y1="33.02" x2="48.26" y2="33.02" width="0.1524" layer="91"/>
-<label x="50.8" y="33.02" size="1.778" layer="95"/>
+<pinref part="TEENSY-41" gate="G$1" pin="30"/>
+<wire x1="7.62" y1="38.1" x2="2.54" y2="38.1" width="0.1524" layer="91"/>
+<label x="-12.7" y="38.1" size="1.778" layer="95"/>
 </segment>
 </net>
 <net name="BUTTON-5-LED" class="0">
-<segment>
-<pinref part="TEENSY-41" gate="G$1" pin="36"/>
-<wire x1="43.18" y1="40.64" x2="48.26" y2="40.64" width="0.1524" layer="91"/>
-<label x="50.8" y="40.64" size="1.778" layer="95"/>
-</segment>
 <segment>
 <wire x1="33.02" y1="-78.74" x2="30.48" y2="-78.74" width="0.1524" layer="91"/>
@@
 <net name="BUTTON-5" class="0">
 <segment>
-<pinref part="TEENSY-41" gate="G$1" pin="35"/>
-<wire x1="43.18" y1="38.1" x2="48.26" y2="38.1" width="0.1524" layer="91"/>
-<label x="50.8" y="38.1" size="1.778" layer="95"/>
-</segment>
-<segment>
 <pinref part="S5" gate="G$1" pin="COM"/>
 <wire x1="38.1" y1="-93.98" x2="35.56" y2="-93.98" width="0.1524" layer="91"/>
 <label x="33.02" y="-93.98" size="1.778" layer="95" rot="R180"/>
 </segment>
+<segment>
+<pinref part="TEENSY-41" gate="G$1" pin="31"/>
+<wire x1="7.62" y1="35.56" x2="2.54" y2="35.56" width="0.1524" layer="91"/>
+<label x="-12.7" y="35.56" size="1.778" layer="95"/>
+</segment>
 </net>
 <net name="BUTTON-6-LED" class="0">
@@
 <label x="78.74" y="-78.74" size="1.778" layer="95" rot="R180"/>
 </segment>
-<segment>
-<pinref part="TEENSY-41" gate="G$1" pin="38"/>
-<wire x1="43.18" y1="45.72" x2="48.26" y2="45.72" width="0.1524" layer="91"/>
-<label x="50.8" y="45.72" size="1.778" layer="95"/>
-</segment>
 </net>
 <net name="BUTTON-6" class="0">
@@
 </segment>
 <segment>
-<pinref part="TEENSY-41" gate="G$1" pin="37"/>
-<wire x1="43.18" y1="43.18" x2="48.26" y2="43.18" width="0.1524" layer="91"/>
-<label x="50.8" y="43.18" size="1.778" layer="95"/>
-</segment>
-</net>
+<pinref part="TEENSY-41" gate="G$1" pin="32"/>
+<wire x1="7.62" y1="33.02" x2="2.54" y2="33.02" width="0.1524" layer="91"/>
+<label x="-12.7" y="33.02" size="1.778" layer="95"/>
+</segment>
+</net>

Commit message: Refactor, add button LEDs
Connections:
- new net N$1: TEENSY-41G$1.39
- net BUTTON-1-LED: now also TEENSY-41G$1.10
- net BUTTON-2-LED: now also TEENSY-41G$1.11
- net BUTTON-3-LED: now also TEENSY-41G$1.12
- net BUTTON-4-LED: now also TEENSY-41G$1.14
- net BUTTON-5-LED: now also TEENSY-41G$1.15
- net BUTTON-6-LED: now also TEENSY-41G$1.22
Changed lines of the file:
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@@
 <attribute name="VALUE" x="85.09" y="-82.042" size="1.778" layer="96"/>
 </instance>
-<instance part="+3V9" gate="G$1" x="-10.16" y="66.04" smashed="yes">
-<attribute name="VALUE" x="-12.7" y="60.96" size="1.778" layer="96" rot="R90"/>
+<instance part="+3V9" gate="G$1" x="-20.32" y="66.04" smashed="yes">
+<attribute name="VALUE" x="-22.86" y="60.96" size="1.778" layer="96" rot="R90"/>
 </instance>
 <instance part="P+4" gate="1" x="111.76" y="-17.78" smashed="yes">
@@
 <pinref part="TEENSY-41" gate="G$1" pin="3.3V"/>
 <pinref part="+3V9" gate="G$1" pin="+3V3"/>
-<wire x1="-10.16" y1="63.5" x2="-10.16" y2="55.88" width="0.1524" layer="91"/>
-<wire x1="-10.16" y1="55.88" x2="7.62" y2="55.88" width="0.1524" layer="91"/>
+<wire x1="-20.32" y1="63.5" x2="-20.32" y2="55.88" width="0.1524" layer="91"/>
+<wire x1="-20.32" y1="55.88" x2="7.62" y2="55.88" width="0.1524" layer="91"/>
 </segment>
 </net>
@@
 <pinref part="R5" gate="G$1" pin="1"/>
 </segment>
+<segment>
+<pinref part="TEENSY-41" gate="G$1" pin="10"/>
+<wire x1="7.62" y1="63.5" x2="2.54" y2="63.5" width="0.1524" layer="91"/>
+<label x="-17.78" y="63.5" size="1.778" layer="95"/>
+</segment>
 </net>
 <net name="N$5" class="0">
@@
 <label x="20.32" y="-27.94" size="1.778" layer="95" rot="R180"/>
 </segment>
+<segment>
+<pinref part="TEENSY-41" gate="G$1" pin="11"/>
+<wire x1="7.62" y1="60.96" x2="2.54" y2="60.96" width="0.1524" layer="91"/>
+<label x="-17.78" y="60.96" size="1.778" layer="95"/>
+</segment>
 </net>
 <net name="N$6" class="0">
@@
 <pinref part="R7" gate="G$1" pin="1"/>
 <label x="73.66" y="-27.94" size="1.778" layer="95" rot="R180"/>
+</segment>
+<segment>
+<pinref part="TEENSY-41" gate="G$1" pin="12"/>
+<wire x1="7.62" y1="58.42" x2="2.54" y2="58.42" width="0.1524" layer="91"/>
+<label x="-17.78" y="58.42" size="1.778" layer="95"/>
 </segment>
 </net>
@@
 <pinref part="R12" gate="G$1" pin="1"/>
 </segment>
+<segment>
+<pinref part="TEENSY-41" gate="G$1" pin="14"/>
+<wire x1="43.18" y1="60.96" x2="48.26" y2="60.96" width="0.1524" layer="91"/>
+<label x="50.8" y="60.96" size="1.778" layer="95"/>
+</segment>
 </net>
 <net name="BUTTON-4" class="0">
@@
 <label x="25.4" y="-78.74" size="1.778" layer="95" rot="R180"/>
 </segment>
+<segment>
+<pinref part="TEENSY-41" gate="G$1" pin="15"/>
+<wire x1="43.18" y1="63.5" x2="48.26" y2="63.5" width="0.1524" layer="91"/>
+<label x="50.8" y="63.5" size="1.778" layer="95"/>
+</segment>
 </net>
 <net name="BUTTON-5" class="0">
@@
 <pinref part="R14" gate="G$1" pin="1"/>
 <label x="78.74" y="-78.74" size="1.778" layer="95" rot="R180"/>
+</segment>
+<segment>
+<pinref part="TEENSY-41" gate="G$1" pin="22"/>
+<wire x1="43.18" y1="81.28" x2="48.26" y2="81.28" width="0.1524" layer="91"/>
+<label x="50.8" y="81.28" size="1.778" layer="95"/>
 </segment>
 </net>
@@
 </segment>
 </net>
+<net name="N$1" class="0">
+<segment>
+<pinref part="TEENSY-41" gate="G$1" pin="39"/>
+<wire x1="43.18" y1="48.26" x2="48.26" y2="48.26" width="0.1524" layer="91"/>
+</segment>
+</net>
